File: hardware/kicad/TDC7201-Module.kicad_pcb (KiCad board)
At the start: 4 copper layers, 80 x 50 mm, 41 parts, among them J1 SMA_PPS_IN, J2 SMA_10MHZ_IN, J3 SMA_WiFi_ANT, J4 USB-C, U1 AMS1117-3.3, U3 TDC7201, U4 TLV3501, U5 TLV3501, U6 TL07401, U7 ESP32-C3-WROOM-02U-N4

Commit message: Fix ferrite bead pad net assignments (L1/L2: +5V→+3V3)
Agent-Logs-Url: https://github.com/jeffkarney/TDC7201-GPSDO-Module/sessions/249e8e96-76a3-4c3b-a7cb-0897e226d90f

Co-authored-by: jeffkarney <201882+jeffkarney@users.noreply.github.com>
Connections:
- L1 pad 2: +5V -> +3V3
- L2 pad 2: +5V -> +3V3
Changed lines of the file:
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@@
     )
       (pad "1" smd rect (at -0.800 0.000) (size 1.20 0.80) (layers "F.Cu" "F.Paste" "F.Mask") (net 3 "+5V"))
-      (pad "2" smd rect (at 0.800 0.000) (size 1.20 0.80) (layers "F.Cu" "F.Paste" "F.Mask") (net 3 "+5V"))
+      (pad "2" smd rect (at 0.800 0.000) (size 1.20 0.80) (layers "F.Cu" "F.Paste" "F.Mask") (net 2 "+3V3"))
   )
   (footprint "Inductor_SMD:L_0805_2012Metric" (layer "F.Cu")
@@
     )
       (pad "1" smd rect (at -0.800 0.000) (size 1.20 0.80) (layers "F.Cu" "F.Paste" "F.Mask") (net 3 "+5V"))
-      (pad "2" smd rect (at 0.800 0.000) (size 1.20 0.80) (layers "F.Cu" "F.Paste" "F.Mask") (net 3 "+5V"))
+      (pad "2" smd rect (at 0.800 0.000) (size 1.20 0.80) (layers "F.Cu" "F.Paste" "F.Mask") (net 2 "+3V3"))
   )
   (footprint "Resistor_SMD:R_0603_1608Metric" (layer "F.Cu")
